Commit message: rename file to add custom parts to kobuki model

File: simulation/kobuki_parts/custom_part.xacro (robot description, xacro)
@@ -1,6 +1,6 @@
 <?xml version="1.0"?>
 <robot xmlns:xacro="http://www.ros.org/wiki/xacro">
-<!-- Front Laser -->
-<xacro:macro name="laser" params="name parent xyz rpy meshes" >
+<!-- custom part -->
+<xacro:macro name="custom_part" params="name parent xyz rpy uriheader part" >
   <joint name="${parent}_${name}_joint" type="fixed">
       <axis xyz="0 0 1" />
@@ -19,5 +19,5 @@
         <origin xyz="0 0 0" rpy="0 0 0"/>
         <geometry>
-          <mesh filename="${meshes}/hokuyo.dae"/>
+          <mesh filename="${uriheader}/${part}.dae"/>
         </geometry>
       </visual>

Commit message: custom_part.xacro: fix collision geometry

File: simulation/kobuki_parts/custom_part.xacro (robot description, xacro)
@@ -13,5 +13,5 @@
         <origin xyz="0 0 0" rpy="0 0 0"/>
         <geometry>
-          <box size="0.1 0.1 0.1"/>
+          <mesh filename="${uriheader}/${part}.dae"/>
         </geometry>
       </collision>
